Commit message: dependencies

File: quadruped_gazebo/urdf/a1/a1_rs.urdf (robot description, URDF)
Before this commit: robot a1_description, 23 links, 22 joints
Links:
- removed link base_link
- added link base; visual box size=0.001 0.001 0.001
Joints:
- joint floating_base: parent base_link -> base

File: quadruped_gazebo/urdf/depth_sensor.urdf.xacro (robot description, xacro)
@@ -1,5 +1,5 @@
 <robot xmlns:xacro="http://ros.org/wiki/xacro">
   <xacro:property name="M_PI" value="3.1415926535897931" />
-  <xacro:macro name="depth_sensor" params="*origin camera_link:=camera_link camera_name:=camera">
+  <xacro:macro name="depth_sensor" params="*origin camera_link:=camera_link camera_name:=camera parent:=base">
     <link name="${camera_link}">
       <visual>
@@ -37,6 +37,6 @@
       </visual>
     </gazebo>rgb(213,28,40)
-    <joint name="${camera_name}_to_base_link" type="fixed">
-      <parent link="base_link"/>
+    <joint name="${camera_name}_to_${parent}" type="fixed">
+      <parent link="${parent}"/>
       <child link="${camera_link}"/>
       <xacro:insert_block name="origin" />
